Commit message: :zap: Update

File: ROS2/packages/robot_description/urdf/ForkliftE.urdf (robot description, URDF)
Before this commit: robot forklift_c, 8 links, 7 joints
Links:
- removed link SM_Forklift_C01_01
- added link ForkliftE; collision mesh filename=file:///home/avent/Documents/ROS2/CageStack_IBVS/packages/r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 scale=1. 1. 1.; collision mesh filename=file:///home/avent/Documents/ROS2/CageStack_IBVS/packages/r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 scale=1. 1. 1.
- added link left_camera_SG3S_ISX031C_GMSL2F_H190XA_01
- added link right_camera_SG3S_ISX031C_GMSL2F_H190XA_01
- link left_back_wheel: geometry visual mesh filename=file:///home/avent/Documents/ROS2/CageStack_IBVS/packages/r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 scale=1. 1. 1.
- link left_front_wheel: geometry visual mesh filename=file:///home/avent/Documents/ROS2/CageStack_IBVS/packages/r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 scale=1. 1. 1.
- link lift: geometry collision mesh filename=file:///home/avent/Documents/ROS2/CageStack_IBVS/packages/r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 scale=1. 1. 1.; collision mesh filename=file:///home/avent/Documents/ROS2/CageStack_IBVS/packages/r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 scale=1. 1. 1.
- link right_back_wheel: geometry visual mesh filename=file:///home/avent/Documents/ROS2/CageStack_IBVS/packages/r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 scale=1. 1. 1.
- link right_front_wheel: geometry visual mesh filename=file:///home/avent/Documents/ROS2/CageStack_IBVS/packages/r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 scale=1. 1. 1.
Joints:
- added joint joint_lift-left_camera_SG3S_ISX031C_GMSL2F_H190XA_01: type fixed, parent lift, child left_camera_SG3S_ISX031C_GMSL2F_H190XA_01, origin xyz=0.6 -0.66 0.09 rpy=1.5707964 0. -2.3561945
- added joint joint_lift-right_camera_SG3S_ISX031C_GMSL2F_H190XA_01: type fixed, parent lift, child right_camera_SG3S_ISX031C_GMSL2F_H190XA_01, origin xyz=-0.6 -0.66 0.09 rpy=1.5707964 0. 2.3561945
- joint left_front_wheel_joint: parent SM_Forklift_C01_01 -> ForkliftE
- joint left_rotator_joint: parent SM_Forklift_C01_01 -> ForkliftE
- joint lift_joint: limit lower=0. upper=2. effort=10000000. velocity=0. -> lower=0. upper=20. effort=10000000. velocity=0.; parent SM_Forklift_C01_01 -> ForkliftE
- joint right_front_wheel_joint: parent SM_Forklift_C01_01 -> ForkliftE
- joint right_rotator_joint: parent SM_Forklift_C01_01 -> ForkliftE

Commit message: :zap: Update

File: ROS2/packages/robot_description/urdf/ForkliftE.urdf (robot description, URDF)
Before this commit: robot ForkliftE_sensors, 10 links, 9 joints
Links:
- removed link ForkliftE
- removed link left_camera_SG3S_ISX031C_GMSL2F_H190XA_01
- removed link right_camera_SG3S_ISX031C_GMSL2F_H190XA_01
- added link SM_Forklift_C01_01; collision mesh filename=file:///home/vn/Documents/MyDrawft/CageStack_IBVS/ROS2/pack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 scale=1. 1. 1.; collision mesh filename=file:///home/vn/Documents/MyDrawft/CageStack_IBVS/ROS2/pack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 scale=1. 1. 1.
- link left_back_wheel: geometry visual mesh filename=file:///home/vn/Documents/MyDrawft/CageStack_IBVS/ROS2/pack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 scale=1. 1. 1.
- link left_front_wheel: geometry visual mesh filename=file:///home/vn/Documents/MyDrawft/CageStack_IBVS/ROS2/pack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 scale=1. 1. 1.
- link left_rotator: geometry collision mesh filename=file:///home/vn/Documents/MyDrawft/CageStack_IBVS/ROS2/pack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 scale=1. 1. 1.; visual mesh filename=file:///home/vn/Documents/MyDrawft/CageStack_IBVS/ROS2/pack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 scale=1. 1. 1.
- link lift: geometry collision mesh filename=file:///home/vn/Documents/MyDrawft/CageStack_IBVS/ROS2/pack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 scale=1. 1. 1.; collision mesh filename=file:///home/vn/Documents/MyDrawft/CageStack_IBVS/ROS2/pack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 scale=1. 1. 1.
- link right_back_wheel: geometry visual mesh filename=file:///home/vn/Documents/MyDrawft/CageStack_IBVS/ROS2/pack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 scale=1. 1. 1.
- link right_front_wheel: geometry visual mesh filename=file:///home/vn/Documents/MyDrawft/CageStack_IBVS/ROS2/pack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 scale=1. 1. 1.
- link right_rotator: geometry collision mesh filename=file:///home/vn/Documents/MyDrawft/CageStack_IBVS/ROS2/pack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 scale=1. 1. 1.; visual mesh filename=file:///home/vn/Documents/MyDrawft/CageStack_IBVS/ROS2/pack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 scale=1. 1. 1.
Joints:
- removed joint joint_lift-left_camera_SG3S_ISX031C_GMSL2F_H190XA_01
- removed joint joint_lift-right_camera_SG3S_ISX031C_GMSL2F_H190XA_01
- joint left_front_wheel_joint: parent ForkliftE -> SM_Forklift_C01_01
- joint left_rotator_joint: parent ForkliftE -> SM_Forklift_C01_01
- joint lift_joint: limit lower=0. upper=20. effort=10000000. velocity=0. -> lower=0. upper=2. effort=10000000. velocity=0.; parent ForkliftE -> SM_Forklift_C01_01
- joint right_front_wheel_joint: parent ForkliftE -> SM_Forklift_C01_01
- joint right_rotator_joint: parent ForkliftE -> SM_Forklift_C01_01

Commit message: :zap: Update

File: ROS2/packages/robot_description/urdf/ForkliftE.urdf (robot description, URDF)
Before this commit: robot forklift_c, 8 links, 7 joints
Links:
- removed link SM_Forklift_C01_01
- added link ForkliftE; collision mesh filename=file:///home/avent/Documents/ROS2/CageStack_IBVS/ROS2/packa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 scale=1. 1. 1.; collision mesh filename=file:///home/avent/Documents/ROS2/CageStack_IBVS/ROS2/packa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 scale=1. 1. 1.
- link left_back_wheel: geometry visual mesh filename=file:///home/avent/Documents/ROS2/CageStack_IBVS/ROS2/packa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 scale=1. 1. 1.
- link left_front_wheel: geometry visual mesh filename=file:///home/avent/Documents/ROS2/CageStack_IBVS/ROS2/packa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 scale=1. 1. 1.
- link left_rotator: geometry collision mesh filename=file:///home/avent/Documents/ROS2/CageStack_IBVS/ROS2/packa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 scale=1. 1. 1.; visual mesh filename=file:///home/avent/Documents/ROS2/CageStack_IBVS/ROS2/packa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 scale=1. 1. 1.
- link lift: geometry collision mesh filename=file:///home/avent/Documents/ROS2/CageStack_IBVS/ROS2/packa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 scale=1. 1. 1.; collision mesh filename=file:///home/avent/Documents/ROS2/CageStack_IBVS/ROS2/packa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 scale=1. 1. 1.
- link right_back_wheel: geometry visual mesh filename=file:///home/avent/Documents/ROS2/CageStack_IBVS/ROS2/packa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 scale=1. 1. 1.
- link right_front_wheel: geometry visual mesh filename=file:///home/avent/Documents/ROS2/CageStack_IBVS/ROS2/packa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 scale=1. 1. 1.
- link right_rotator: geometry collision mesh filename=file:///home/avent/Documents/ROS2/CageStack_IBVS/ROS2/packa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 scale=1. 1. 1.; visual mesh filename=file:///home/avent/Documents/ROS2/CageStack_IBVS/ROS2/packa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 scale=1. 1. 1.
Joints:
- joint left_front_wheel_joint: origin xyz=0.2687796 0.5974939 0.3251018 rpy=0. 0. 1.5707964 -> xyz=0.2687795 0.5976231 0.4326027 rpy=0. 0. 1.5707964; parent SM_Forklift_C01_01 -> ForkliftE
- joint left_rotator_joint: origin xyz=-1.385914 0.4061331 0.2102286 rpy=0. 0. 1.5707964 -> xyz=-1.385914 0.4062623 0.3177295 rpy=0. 0. 1.5707964; parent SM_Forklift_C01_01 -> ForkliftE
- joint lift_joint: origin xyz=0. 0. 0. rpy=0. 0. 1.5707964 -> xyz=-0. 0.0001292 0.1075009 rpy=0. 0. 1.5707964; parent SM_Forklift_C01_01 -> ForkliftE
- joint right_front_wheel_joint: origin xyz=0.2687802 -0.59744 0.3251018 rpy=0. 0. 1.5707964 -> xyz=0.2687801 -0.5973108 0.4326027 rpy=0. 0. 1.5707964; parent SM_Forklift_C01_01 -> ForkliftE
- joint right_rotator_joint: origin xyz=-1.385914 -0.406132 0.2102286 rpy=0. 0. 1.5707964 -> xyz=-1.385914 -0.4060028 0.3177295 rpy=0. 0. 1.5707964; parent SM_Forklift_C01_01 -> ForkliftE

Commit message: :zap: Update

File: ROS2/packages/robot_description/urdf/ForkliftE.urdf (robot description, URDF)
Before this commit: robot , 8 links, 7 joints
Links:
- removed link ForkliftE
- added link SM_Forklift_C01_01; collision mesh filename=file:///home/vn/Documents/MyDrawft/CageStack_IBVS/ROS2/pack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 scale=1. 1. 1.; collision mesh filename=file:///home/vn/Documents/MyDrawft/CageStack_IBVS/ROS2/pack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 scale=1. 1. 1.
- link left_back_wheel: geometry visual mesh filename=file:///home/vn/Documents/MyDrawft/CageStack_IBVS/ROS2/pack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 scale=1. 1. 1.
- link left_front_wheel: geometry visual mesh filename=file:///home/vn/Documents/MyDrawft/CageStack_IBVS/ROS2/pack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 scale=1. 1. 1.
- link left_rotator: geometry collision mesh filename=file:///home/vn/Documents/MyDrawft/CageStack_IBVS/ROS2/pack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 scale=1. 1. 1.; visual mesh filename=file:///home/vn/Documents/MyDrawft/CageStack_IBVS/ROS2/pack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 scale=1. 1. 1.
- link lift: geometry collision mesh filename=file:///home/vn/Documents/MyDrawft/CageStack_IBVS/ROS2/pack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 scale=1. 1. 1.; collision mesh filename=file:///home/vn/Documents/MyDrawft/CageStack_IBVS/ROS2/pack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 scale=1. 1. 1.
- link right_back_wheel: geometry visual mesh filename=file:///home/vn/Documents/MyDrawft/CageStack_IBVS/ROS2/pack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 scale=1. 1. 1.
- link right_front_wheel: geometry visual mesh filename=file:///home/vn/Documents/MyDrawft/CageStack_IBVS/ROS2/pack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 scale=1. 1. 1.
- link right_rotator: geometry collision mesh filename=file:///home/vn/Documents/MyDrawft/CageStack_IBVS/ROS2/pack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 scale=1. 1. 1.; visual mesh filename=file:///home/vn/Documents/MyDrawft/CageStack_IBVS/ROS2/pack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 scale=1. 1. 1.
Joints:
- joint left_front_wheel_joint: origin xyz=0.2687795 0.5976231 0.4326027 rpy=0. 0. 1.5707964 -> xyz=0.2687796 0.5974939 0.3251018 rpy=0. 0. 1.5707964; parent ForkliftE -> SM_Forklift_C01_01
- joint left_rotator_joint: origin xyz=-1.385914 0.4062623 0.3177295 rpy=0. 0. 1.5707964 -> xyz=-1.385914 0.4061331 0.2102286 rpy=0. 0. 1.5707964; parent ForkliftE -> SM_Forklift_C01_01
- joint lift_joint: origin xyz=-0. 0.0001292 0.1075009 rpy=0. 0. 1.5707964 -> xyz=0. 0. 0. rpy=0. 0. 1.5707964; parent ForkliftE -> SM_Forklift_C01_01
- joint right_front_wheel_joint: origin xyz=0.2687801 -0.5973108 0.4326027 rpy=0. 0. 1.5707964 -> xyz=0.2687802 -0.59744 0.3251018 rpy=0. 0. 1.5707964; parent ForkliftE -> SM_Forklift_C01_01
- joint right_rotator_joint: origin xyz=-1.385914 -0.4060028 0.3177295 rpy=0. 0. 1.5707964 -> xyz=-1.385914 -0.406132 0.2102286 rpy=0. 0. 1.5707964; parent ForkliftE -> SM_Forklift_C01_01
